File: Clock.kicad_sch (KiCad schematic)
At the start: 8 parts, among them U4 LM555xM

Commit message: Removido o circuito debounce do dipswitch
Parts:
- C1: renamed from C19; footprint (none) -> Capacitor_THT:CP_Radial_D4.0mm_P2.00mm
- C2: renamed from C20; value 0.01uF -> 10nF; footprint (none) -> Capacitor_THT:C_Rect_L4.6mm_W3.0mm_P2.50mm_MKS02_FKP02
- R22: renamed from R41; footprint (none) -> Resistor_THT:R_Axial_DIN0207_L6.3mm_D2.5mm_P7.62mm_Horizontal
- R23: renamed from R42; footprint (none) -> Resistor_THT:R_Axial_DIN0207_L6.3mm_D2.5mm_P7.62mm_Horizontal
- R24: renamed from R43; footprint (none) -> Resistor_THT:R_Axial_DIN0207_L6.3mm_D2.5mm_P7.62mm_Horizontal
- R25: renamed from R44; footprint (none) -> Resistor_THT:R_Axial_DIN0207_L6.3mm_D2.5mm_P7.62mm_Horizontal
- RV1: footprint (none) -> Potentiometer_THT:Potentiometer_Alps_RK09K_Single_Horizontal
- U1: renamed from U4; footprint Package_SO:SOIC-8_3.9x4.9mm_P1.27mm -> Package_DIP:DIP-8_W7.62mm_Socket
Changed lines of the file:
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@@
   (symbol (lib_id "Device:R") (at 180.34 95.25 90) (unit 1)
     (in_bom yes) (on_board yes)
-    (property "Reference" "R42" (id 0) (at 180.34 92.71 90))
+    (property "Reference" "R23" (id 0) (at 180.34 92.71 90))
     (property "Value" "1K" (id 1) (at 180.34 95.25 90))
-    (property "Footprint" "" (id 2) (at 180.34 97.028 90)
+    (property "Footprint" "Resistor_THT:R_Axial_DIN0207_L6.3mm_D2.5mm_P7.62mm_Horizontal" (id 2) (at 180.34 97.028 90)
       (effects (font (size 1.27 1.27)) hide)
     )
@@
   (symbol (lib_id "power:+5V") (at 115.57 100.33 0) (unit 1)
     (in_bom yes) (on_board yes) (fields_autoplaced)
-    (property "Reference" "#PWR054" (id 0) (at 115.57 104.14 0)
+    (property "Reference" "#PWR013" (id 0) (at 115.57 104.14 0)
       (effects (font (size 1.27 1.27)) hide)
     )
@@
   (symbol (lib_id "power:GND") (at 132.08 109.22 0) (unit 1)
     (in_bom yes) (on_board yes) (fields_autoplaced)
-    (property "Reference" "#PWR056" (id 0) (at 132.08 115.57 0)
+    (property "Reference" "#PWR015" (id 0) (at 132.08 115.57 0)
       (effects (font (size 1.27 1.27)) hide)
     )
@@
   (symbol (lib_id "power:+5V") (at 132.08 74.93 0) (unit 1)
     (in_bom yes) (on_board yes) (fields_autoplaced)
-    (property "Reference" "#PWR055" (id 0) (at 132.08 78.74 0)
+    (property "Reference" "#PWR014" (id 0) (at 132.08 78.74 0)
       (effects (font (size 1.27 1.27)) hide)
     )
@@
   (symbol (lib_id "power:GND") (at 88.9 110.49 0) (unit 1)
     (in_bom yes) (on_board yes)
-    (property "Reference" "#PWR052" (id 0) (at 88.9 116.84 0)
+    (property "Reference" "#PWR011" (id 0) (at 88.9 116.84 0)
       (effects (font (size 1.27 1.27)) hide)
     )
@@
   (symbol (lib_id "Device:C_Polarized") (at 88.9 102.87 0) (unit 1)
     (in_bom yes) (on_board yes) (fields_autoplaced)
-    (property "Reference" "C19" (id 0) (at 91.821 101.0725 0)
+    (property "Reference" "C1" (id 0) (at 91.821 101.0725 0)
       (effects (font (size 1.27 1.27)) (justify left))
     )
@@
       (effects (font (size 1.27 1.27)) (justify left))
     )
-    (property "Footprint" "" (id 2) (at 89.8652 106.68 0)
+    (property "Footprint" "Capacitor_THT:CP_Radial_D4.0mm_P2.00mm" (id 2) (at 89.8652 106.68 0)
       (effects (font (size 1.27 1.27)) hide)
     )
@@
       (effects (font (size 1.27 1.27)) (justify right))
     )
-    (property "Footprint" "" (id 2) (at 190.5 95.25 0)
+    (property "Footprint" "Potentiometer_THT:Potentiometer_Alps_RK09K_Single_Horizontal" (id 2) (at 190.5 95.25 0)
       (effects (font (size 1.27 1.27)) hide)
     )
@@
   (symbol (lib_id "Timer:LM555xM") (at 132.08 95.25 0) (unit 1)
     (in_bom yes) (on_board yes) (fields_autoplaced)
-    (property "Reference" "U4" (id 0) (at 134.0994 83.6635 0)
+    (property "Reference" "U1" (id 0) (at 134.0994 83.6635 0)
       (effects (font (size 1.27 1.27)) (justify left))
     )
@@
       (effects (font (size 1.27 1.27)) (justify left))
     )
-    (property "Footprint" "Package_SO:SOIC-8_3.9x4.9mm_P1.27mm" (id 2) (at 153.67 105.41 0)
+    (property "Footprint" "Package_DIP:DIP-8_W7.62mm_Socket" (id 2) (at 153.67 105.41 0)
       (effects (font (size 1.27 1.27)) hide)
     )
@@
   (symbol (lib_id "power:GND") (at 105.41 110.49 0) (unit 1)
     (in_bom yes) (on_board yes)
-    (property "Reference" "#PWR053" (id 0) (at 105.41 116.84 0)
+    (property "Reference" "#PWR012" (id 0) (at 105.41 116.84 0)
       (effects (font (size 1.27 1.27)) hide)
     )
@@
   (symbol (lib_id "Device:C") (at 105.41 102.87 0) (unit 1)
     (in_bom yes) (on_board yes) (fields_autoplaced)
-    (property "Reference" "C20" (id 0) (at 108.331 101.9615 0)
-      (effects (font (size 1.27 1.27)) (justify left))
-    )
-    (property "Value" "0.01uF" (id 1) (at 108.331 104.7366 0)
-      (effects (font (size 1.27 1.27)) (justify left))
-    )
-    (property "Footprint" "" (id 2) (at 106.3752 106.68 0)
+    (property "Reference" "C2" (id 0) (at 108.331 101.9615 0)
+      (effects (font (size 1.27 1.27)) (justify left))
+    )
+    (property "Value" "10nF" (id 1) (at 108.331 104.7366 0)
+      (effects (font (size 1.27 1.27)) (justify left))
+    )
+    (property "Footprint" "Capacitor_THT:C_Rect_L4.6mm_W3.0mm_P2.50mm_MKS02_FKP02" (id 2) (at 106.3752 106.68 0)
       (effects (font (size 1.27 1.27)) hide)
     )
@@
   (symbol (lib_id "power:+5V") (at 170.18 78.74 0) (unit 1)
     (in_bom yes) (on_board yes) (fields_autoplaced)
-    (property "Reference" "#PWR057" (id 0) (at 170.18 82.55 0)
+    (property "Reference" "#PWR016" (id 0) (at 170.18 82.55 0)
       (effects (font (size 1.27 1.27)) hide)
     )
@@
   (symbol (lib_id "Device:R") (at 170.18 86.36 0) (unit 1)
     (in_bom yes) (on_board yes)
-    (property "Reference" "R41" (id 0) (at 171.958 85.4515 0)
+    (property "Reference" "R22" (id 0) (at 171.958 85.4515 0)
       (effects (font (size 1.27 1.27)) (justify left))
     )
@@
       (effects (font (size 1.27 1.27)) (justify left))
     )
-    (property "Footprint" "" (id 2) (at 168.402 86.36 90)
+    (property "Footprint" "Resistor_THT:R_Axial_DIN0207_L6.3mm_D2.5mm_P7.62mm_Horizontal" (id 2) (at 168.402 86.36 90)
       (effects (font (size 1.27 1.27)) hide)
     )
@@
   (symbol (lib_id "Device:R") (at 198.12 74.93 180) (unit 1)
     (in_bom yes) (on_board yes)
-    (property "Reference" "R44" (id 0) (at 199.898 74.0215 0)
+    (property "Reference" "R25" (id 0) (at 199.898 74.0215 0)
       (effects (font (size 1.27 1.27)) (justify right))
     )
@@
       (effects (font (size 1.27 1.27)) (justify right))
     )
-    (property "Footprint" "" (id 2) (at 199.898 74.93 90)
+    (property "Footprint" "Resistor_THT:R_Axial_DIN0207_L6.3mm_D2.5mm_P7.62mm_Horizontal" (id 2) (at 199.898 74.93 90)
       (effects (font (size 1.27 1.27)) hide)
     )
@@
   (symbol (lib_id "power:GND") (at 198.12 82.55 0) (unit 1)
     (in_bom yes) (on_board yes)
-    (property "Reference" "#PWR058" (id 0) (at 198.12 88.9 0)
+    (property "Reference" "#PWR017" (id 0) (at 198.12 88.9 0)
       (effects (font (size 1.27 1.27)) hide)
     )
@@
   (symbol (lib_id "Device:R") (at 185.42 68.58 90) (unit 1)
     (in_bom yes) (on_board yes)
-    (property "Reference" "R43" (id 0) (at 185.42 66.04 90))
+    (property "Reference" "R24" (id 0) (at 185.42 66.04 90))
     (property "Value" "10k" (id 1) (at 185.42 68.58 90))
-    (property "Footprint" "" (id 2) (at 185.42 70.358 90)
-      (effects (font (size 1.27 1.27)) hide)
-    )
+    (property "Footprint" "Resistor_THT:R_Axial_DIN0207_L6.3mm_D2.5mm_P7.62mm_Horizontal" (id 2) (at 185.42 70.358 90)
+      (effects (font (size 1.27 1.27)) hide)
+    )

Commit message: Adicionado os furos de montagem. Definidos os footprints
Parts:
- RV1: footprint Potentiometer_THT:Potentiometer_Alps_RK09K_Single_Horizontal -> Potentiometer_THT:Potentiometer_Alps_RK163_Single_Horizontal
Changed lines of the file:
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@@
       (effects (font (size 1.27 1.27)) (justify right))
     )
-    (property "Footprint" "Potentiometer_THT:Potentiometer_Alps_RK09K_Single_Horizontal" (id 2) (at 190.5 95.25 0)
+    (property "Footprint" "Potentiometer_THT:Potentiometer_Alps_RK163_Single_Horizontal" (id 2) (at 190.5 95.25 0)
       (effects (font (size 1.27 1.27)) hide)
     )

Commit message: Corrigido o footprint dos capacitores. Adicionado um capacitor de bypass. Adicionado o ground plane e logo.
Parts:
- added C10: 10uF, Capacitor_THT:CP_Radial_D4.0mm_P2.00mm, symbol Device:C_Polarized
- C1: value 1uF -> 10uF
- C2: footprint Capacitor_THT:C_Rect_L4.6mm_W3.0mm_P2.50mm_MKS02_FKP02 -> Capacitor_THT:C_Rect_L7.0mm_W3.5mm_P5.00mm
Connections:
- net +5V: now also C10.1
- net GND: now also C10.2
Changed lines of the file:
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@@
   (junction (at 198.12 68.58) (diameter 0) (color 0 0 0 0)
   )
+  (junction (at 132.08 69.85) (diameter 0) (color 0 0 0 0)
+  )
   (junction (at 149.86 118.11) (diameter 0) (color 0 0 0 0)
   )
@@
   )
   (no_connect (at 190.5 91.44))
-  (wire (pts (xy 132.08 74.93) (xy 132.08 85.09))
+  (wire (pts (xy 132.08 67.31) (xy 132.08 69.85))
     (stroke (width 0) (type default) (color 0 0 0 0))
   )
@@
     (stroke (width 0) (type default) (color 0 0 0 0))
   )
+  (wire (pts (xy 118.11 72.39) (xy 118.11 69.85))
+    (stroke (width 0) (type default) (color 0 0 0 0))
+  )
+  (wire (pts (xy 118.11 80.01) (xy 118.11 81.28))
+    (stroke (width 0) (type default) (color 0 0 0 0))
+  )
   (wire (pts (xy 144.78 100.33) (xy 149.86 100.33))
     (stroke (width 0) (type default) (color 0 0 0 0))
@@
     (stroke (width 0) (type default) (color 0 0 0 0))
   )
+  (wire (pts (xy 132.08 69.85) (xy 132.08 85.09))
+    (stroke (width 0) (type default) (color 0 0 0 0))
+  )
   (wire (pts (xy 144.78 90.17) (xy 157.48 90.17))
     (stroke (width 0) (type default) (color 0 0 0 0))
@@
   )
   (wire (pts (xy 198.12 68.58) (xy 213.36 68.58))
+    (stroke (width 0) (type default) (color 0 0 0 0))
+  )
+  (wire (pts (xy 118.11 69.85) (xy 132.08 69.85))
     (stroke (width 0) (type default) (color 0 0 0 0))
   )
@@
     (pin "1")
   )
+  (symbol (lib_id "power:GND") (at 118.11 81.28 0) (unit 1)
+    (in_bom yes) (on_board yes)
+    (property "Reference" "#PWR0101" (id 0) (at 118.11 87.63 0)
+      (effects (font (size 1.27 1.27)) hide)
+    )
+    (property "Value" "GND" (id 1) (at 118.11 85.8425 0))
+    (property "Footprint" "" (id 2) (at 118.11 81.28 0)
+      (effects (font (size 1.27 1.27)) hide)
+    )
+    (property "Datasheet" "" (id 3) (at 118.11 81.28 0)
+      (effects (font (size 1.27 1.27)) hide)
+    )
+    (pin "1")
+  )
   (symbol (lib_id "power:GND") (at 132.08 109.22 0) (unit 1)
     (in_bom yes) (on_board yes) (fields_autoplaced)
@@
     (pin "1")
   )
-  (symbol (lib_id "power:+5V") (at 132.08 74.93 0) (unit 1)
-    (in_bom yes) (on_board yes) (fields_autoplaced)
-    (property "Reference" "#PWR014" (id 0) (at 132.08 78.74 0)
-      (effects (font (size 1.27 1.27)) hide)
-    )
-    (property "Value" "+5V" (id 1) (at 132.08 71.3255 0))
-    (property "Footprint" "" (id 2) (at 132.08 74.93 0)
-      (effects (font (size 1.27 1.27)) hide)
-    )
-    (property "Datasheet" "" (id 3) (at 132.08 74.93 0)
+  (symbol (lib_id "power:+5V") (at 132.08 67.31 0) (unit 1)
+    (in_bom yes) (on_board yes) (fields_autoplaced)
+    (property "Reference" "#PWR014" (id 0) (at 132.08 71.12 0)
+      (effects (font (size 1.27 1.27)) hide)
+    )
+    (property "Value" "+5V" (id 1) (at 132.08 63.7055 0))
+    (property "Footprint" "" (id 2) (at 132.08 67.31 0)
+      (effects (font (size 1.27 1.27)) hide)
+    )
+    (property "Datasheet" "" (id 3) (at 132.08 67.31 0)
       (effects (font (size 1.27 1.27)) hide)
     )
@@
       (effects (font (size 1.27 1.27)) (justify left))
     )
-    (property "Value" "1uF" (id 1) (at 91.821 103.8476 0)
+    (property "Value" "10uF" (id 1) (at 91.821 103.8476 0)
       (effects (font (size 1.27 1.27)) (justify left))
     )
@@
     (pin "7")
   )
+  (symbol (lib_id "Device:C_Polarized") (at 118.11 76.2 0) (unit 1)
+    (in_bom yes) (on_board yes) (fields_autoplaced)
+    (property "Reference" "C10" (id 0) (at 121.92 74.0409 0)
+      (effects (font (size 1.27 1.27)) (justify left))
+    )
+    (property "Value" "10uF" (id 1) (at 121.92 76.5809 0)
+      (effects (font (size 1.27 1.27)) (justify left))
+    )
+    (property "Footprint" "Capacitor_THT:CP_Radial_D4.0mm_P2.00mm" (id 2) (at 119.0752 80.01 0)
+      (effects (font (size 1.27 1.27)) hide)
+    )
+    (property "Datasheet" "~" (id 3) (at 118.11 76.2 0)
+      (effects (font (size 1.27 1.27)) hide)
+    )
+    (pin "1")
+    (pin "2")
+  )
   (symbol (lib_id "power:GND") (at 105.41 110.49 0) (unit 1)
     (in_bom yes) (on_board yes)
@@
       (effects (font (size 1.27 1.27)) (justify left))
     )
-    (property "Footprint" "Capacitor_THT:C_Rect_L4.6mm_W3.0mm_P2.50mm_MKS02_FKP02" (id 2) (at 106.3752 106.68 0)
-      (effects (font (size 1.27 1.27)) hide)
-    )
+    (property "Footprint" "Capacitor_THT:C_Rect_L7.0mm_W3.5mm_P5.00mm" (id 2) (at 106.3752 106.68 0)
+      (effects (font (size 1.27 1.27)) hide)
+    )

Commit message: Atualizado os valores dos capacitores
Parts:
- C1: value 10uF -> 47uF
Changed lines of the file:
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@@
       (effects (font (size 1.27 1.27)) (justify left))
     )
-    (property "Value" "10uF" (id 1) (at 91.821 103.8476 0)
+    (property "Value" "47uF" (id 1) (at 91.821 103.8476 0)
       (effects (font (size 1.27 1.27)) (justify left))
     )
