File: DebounceCircuit.kicad_sch (KiCad schematic)
At the start: 25 parts

Commit message: Adicionado os botões e clock. Adicionada interface com o Analog Discovery 2.
Parts:
- C10, C11, C12, C7, C8, C9: renamed from C?; value C -> 100nF
- R17, R18, R19, R20, R21, R22, R23, R24, R25, R26, R27, R28: renamed from R?; value R -> 10k
- gave numbers to parts that had none: 1
Other:
- company: (none) -> Ailton Luiz Dias Siqueira Junior
- title: (none) -> FPGA Input Board - Debounce Circuit

Commit message: Removido o circuito debounce do dipswitch
Parts:
- C3: renamed from C7; footprint (none) -> Capacitor_THT:C_Rect_L4.6mm_W3.0mm_P2.50mm_MKS02_FKP02
- C4: renamed from C8; footprint (none) -> Capacitor_THT:C_Rect_L4.6mm_W3.0mm_P2.50mm_MKS02_FKP02
- C5: renamed from C9; footprint (none) -> Capacitor_THT:C_Rect_L4.6mm_W3.0mm_P2.50mm_MKS02_FKP02
- C6: renamed from C10; footprint (none) -> Capacitor_THT:C_Rect_L4.6mm_W3.0mm_P2.50mm_MKS02_FKP02
- C7: renamed from C11; footprint (none) -> Capacitor_THT:C_Rect_L4.6mm_W3.0mm_P2.50mm_MKS02_FKP02
- C8: renamed from C12; footprint (none) -> Capacitor_THT:C_Rect_L4.6mm_W3.0mm_P2.50mm_MKS02_FKP02
- R26: renamed from R17; footprint (none) -> Resistor_THT:R_Axial_DIN0207_L6.3mm_D2.5mm_P7.62mm_Horizontal
- R27: renamed from R18; footprint (none) -> Resistor_THT:R_Axial_DIN0207_L6.3mm_D2.5mm_P7.62mm_Horizontal
- R28: renamed from R19; footprint (none) -> Resistor_THT:R_Axial_DIN0207_L6.3mm_D2.5mm_P7.62mm_Horizontal
- R29: renamed from R20; footprint (none) -> Resistor_THT:R_Axial_DIN0207_L6.3mm_D2.5mm_P7.62mm_Horizontal
- R30: renamed from R21; footprint (none) -> Resistor_THT:R_Axial_DIN0207_L6.3mm_D2.5mm_P7.62mm_Horizontal
- R31: renamed from R22; footprint (none) -> Resistor_THT:R_Axial_DIN0207_L6.3mm_D2.5mm_P7.62mm_Horizontal
- R32: renamed from R23; footprint (none) -> Resistor_THT:R_Axial_DIN0207_L6.3mm_D2.5mm_P7.62mm_Horizontal
- R33: renamed from R24; footprint (none) -> Resistor_THT:R_Axial_DIN0207_L6.3mm_D2.5mm_P7.62mm_Horizontal
- R34: renamed from R25; footprint (none) -> Resistor_THT:R_Axial_DIN0207_L6.3mm_D2.5mm_P7.62mm_Horizontal
- R35: renamed from R26; footprint (none) -> Resistor_THT:R_Axial_DIN0207_L6.3mm_D2.5mm_P7.62mm_Horizontal
- R36: renamed from R27; footprint (none) -> Resistor_THT:R_Axial_DIN0207_L6.3mm_D2.5mm_P7.62mm_Horizontal
- R37: renamed from R28; footprint (none) -> Resistor_THT:R_Axial_DIN0207_L6.3mm_D2.5mm_P7.62mm_Horizontal
- U2: footprint (none) -> Package_DIP:DIP-14_W7.62mm_Socket

Commit message: Adicionado os furos de montagem. Definidos os footprints
Connections:
- net +3V3: now also U2.14 (VCC)
- net DBC2: now also U2.4; no longer U2.2
- net DBC3: now also U2.6; no longer U2.2
- net DBC4: now also U2.8; no longer U2.2
- net DBC5: now also U2.10; no longer U2.2
- net DBC6: now also U2.12; no longer U2.2
- net GND: now also U2.7 (GND)
- net at C8.1, R37.2: now also U2.13; no longer U2.1
- net at C5.1, R32.2: now also U2.5; no longer U2.1
- net at C7.1, R36.2: now also U2.11; no longer U2.1
- net at C6.1, R33.2: now also U2.9; no longer U2.1
- net at C4.1, R31.2: now also U2.3; no longer U2.1
Changed lines of the file:
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@@
     (effects (font (size 1.27 1.27)) (justify right))
   )
-  (symbol (lib_id "74xx:74HC14") (at 203.2 82.55 0)
+  (symbol (lib_id "74xx:74HC14") (at 203.2 82.55 0) (unit 6)
     (in_bom yes) (on_board yes) (fields_autoplaced)
     (property "Reference" "U2" (id 0) (at 203.2 73.66 0))
@@
     (pin "13")
   )
-  (symbol (lib_id "power:GND") (at 186.69 62.23 0)
+  (symbol (lib_id "power:GND") (at 186.69 62.23 0) (unit 1)
     (in_bom yes) (on_board yes) (fields_autoplaced)
     (property "Reference" "#PWR030" (id 0) (at 186.69 68.58 0)
@@
     (pin "1")
   )
-  (symbol (lib_id "power:GND") (at 165.1 151.13 0)
+  (symbol (lib_id "power:GND") (at 165.1 151.13 0) (unit 1)
     (in_bom yes) (on_board yes) (fields_autoplaced)
     (property "Reference" "#PWR027" (id 0) (at 165.1 157.48 0)
@@
     (pin "1")
   )
-  (symbol (lib_id "power:GND") (at 99.06 163.83 0)
+  (symbol (lib_id "power:GND") (at 99.06 163.83 0) (unit 1)
     (in_bom yes) (on_board yes) (fields_autoplaced)
     (property "Reference" "#PWR025" (id 0) (at 99.06 170.18 0)
@@
     (pin "1")
   )
-  (symbol (lib_id "power:GND") (at 186.69 97.79 0)
+  (symbol (lib_id "power:GND") (at 186.69 97.79 0) (unit 1)
     (in_bom yes) (on_board yes) (fields_autoplaced)
     (property "Reference" "#PWR031" (id 0) (at 186.69 104.14 0)
@@
     (pin "1")
   )
-  (symbol (lib_id "74xx:74HC14") (at 165.1 133.35 0)
+  (symbol (lib_id "74xx:74HC14") (at 165.1 133.35 0) (unit 7)
     (in_bom yes) (on_board yes) (fields_autoplaced)
     (property "Reference" "U2" (id 0) (at 171.45 132.0799 0)
@@
     (pin "7")
   )
-  (symbol (lib_id "74xx:74HC14") (at 110.49 116.84 0)
+  (symbol (lib_id "74xx:74HC14") (at 110.49 116.84 0) (unit 3)
     (in_bom yes) (on_board yes) (fields_autoplaced)
     (property "Reference" "U2" (id 0) (at 110.49 107.95 0))
@@
     (pin "6")
   )
-  (symbol (lib_id "power:GND") (at 99.06 101.6 0)
+  (symbol (lib_id "power:GND") (at 99.06 101.6 0) (unit 1)
     (in_bom yes) (on_board yes) (fields_autoplaced)
     (property "Reference" "#PWR023" (id 0) (at 99.06 107.95 0)
@@
     (pin "1")
   )
-  (symbol (lib_id "Device:C") (at 186.69 54.61 0)
+  (symbol (lib_id "Device:C") (at 186.69 54.61 0) (unit 1)
     (in_bom yes) (on_board yes) (fields_autoplaced)
     (property "Reference" "C7" (id 0) (at 190.5 53.3399 0)
@@
     (pin "2")
   )
-  (symbol (lib_id "Device:R") (at 168.91 39.37 180)
+  (symbol (lib_id "Device:R") (at 168.91 39.37 180) (unit 1)
     (in_bom yes) (on_board yes) (fields_autoplaced)
     (property "Reference" "R34" (id 0) (at 171.45 38.0999 0)
@@
     (pin "2")
   )
-  (symbol (lib_id "power:+3.3V") (at 80.01 33.02 0)
+  (symbol (lib_id "power:+3.3V") (at 80.01 33.02 0) (unit 1)
     (in_bom yes) (on_board yes) (fields_autoplaced)
     (property "Reference" "#PWR018" (id 0) (at 80.01 36.83 0)
@@
     (pin "1")
   )
-  (symbol (lib_id "power:GND") (at 99.06 132.08 0)
+  (symbol (lib_id "power:GND") (at 99.06 132.08 0) (unit 1)
     (in_bom yes) (on_board yes) (fields_autoplaced)
     (property "Reference" "#PWR024" (id 0) (at 99.06 138.43 0)
@@
     (pin "1")
   )
-  (symbol (lib_id "Device:R") (at 91.44 148.59 90)
+  (symbol (lib_id "Device:R") (at 91.44 148.59 90) (unit 1)
     (in_bom yes) (on_board yes) (fields_autoplaced)
     (property "Reference" "R33" (id 0) (at 91.44 142.24 90))
@@
     (pin "2")
   )
-  (symbol (lib_id "power:GND") (at 97.79 66.04 0)
+  (symbol (lib_id "power:GND") (at 97.79 66.04 0) (unit 1)
     (in_bom yes) (on_board yes) (fields_autoplaced)
     (property "Reference" "#PWR022" (id 0) (at 97.79 72.39 0)
@@
     (pin "1")
   )
-  (symbol (lib_id "74xx:74HC14") (at 203.2 46.99 0)
+  (symbol (lib_id "74xx:74HC14") (at 203.2 46.99 0) (unit 5)
     (in_bom yes) (on_board yes)
     (property "Reference" "U2" (id 0) (at 203.2 38.1 0))
@@
     (pin "11")
   )
-  (symbol (lib_id "Device:R") (at 168.91 74.93 180)
+  (symbol (lib_id "Device:R") (at 168.91 74.93 180) (unit 1)
     (in_bom yes) (on_board yes) (fields_autoplaced)
     (property "Reference" "R35" (id 0) (at 171.45 73.6599 0)
@@
     (pin "2")
   )
-  (symbol (lib_id "Device:C") (at 186.69 90.17 0)
+  (symbol (lib_id "Device:C") (at 186.69 90.17 0) (unit 1)
     (in_bom yes) (on_board yes) (fields_autoplaced)
     (property "Reference" "C8" (id 0) (at 190.5 88.8999 0)
@@
     (pin "2")
   )
-  (symbol (lib_id "Device:R") (at 90.17 50.8 90)
+  (symbol (lib_id "Device:R") (at 90.17 50.8 90) (unit 1)
     (in_bom yes) (on_board yes) (fields_autoplaced)
     (property "Reference" "R30" (id 0) (at 90.17 44.45 90))
@@
     (pin "2")
   )
-  (symbol (lib_id "Device:R") (at 91.44 86.36 90)
+  (symbol (lib_id "Device:R") (at 91.44 86.36 90) (unit 1)
     (in_bom yes) (on_board yes) (fields_autoplaced)
     (property "Reference" "R31" (id 0) (at 91.44 80.01 90))
@@
     (pin "2")
   )
-  (symbol (lib_id "power:+3.3V") (at 81.28 99.06 0)
+  (symbol (lib_id "power:+3.3V") (at 81.28 99.06 0) (unit 1)
     (in_bom yes) (on_board yes) (fields_autoplaced)
     (property "Reference" "#PWR020" (id 0) (at 81.28 102.87 0)
@@
     (pin "1")
   )
-  (symbol (lib_id "Device:R") (at 80.01 43.18 180)
+  (symbol (lib_id "Device:R") (at 80.01 43.18 180) (unit 1)
     (in_bom yes) (on_board yes) (fields_autoplaced)
     (property "Reference" "R26" (id 0) (at 82.55 41.9099 0)
@@
     (pin "2")
   )
-  (symbol (lib_id "Device:C") (at 99.06 156.21 0)
+  (symbol (lib_id "Device:C") (at 99.06 156.21 0) (unit 1)
     (in_bom yes) (on_board yes) (fields_autoplaced)
     (property "Reference" "C6" (id 0) (at 102.87 154.9399 0)
@@
     (pin "2")
   )
-  (symbol (lib_id "Device:R") (at 81.28 78.74 180)
+  (symbol (lib_id "Device:R") (at 81.28 78.74 180) (unit 1)
     (in_bom yes) (on_board yes) (fields_autoplaced)
     (property "Reference" "R27" (id 0) (at 83.82 77.4699 0)
@@
     (pin "2")
   )
-  (symbol (lib_id "power:+3.3V") (at 168.91 64.77 0)
+  (symbol (lib_id "power:+3.3V") (at 168.91 64.77 0) (unit 1)
     (in_bom yes) (on_board yes) (fields_autoplaced)
     (property "Reference" "#PWR029" (id 0) (at 168.91 68.58 0)
@@
     (pin "1")
   )
-  (symbol (lib_id "Device:R") (at 179.07 46.99 90)
+  (symbol (lib_id "Device:R") (at 179.07 46.99 90) (unit 1)
     (in_bom yes) (on_board yes) (fields_autoplaced)
     (property "Reference" "R36" (id 0) (at 179.07 40.64 90))
@@
     (pin "2")
   )
-  (symbol (lib_id "74xx:74HC14") (at 110.49 148.59 0)
+  (symbol (lib_id "74xx:74HC14") (at 110.49 148.59 0) (unit 4)
     (in_bom yes) (on_board yes) (fields_autoplaced)
     (property "Reference" "U2" (id 0) (at 110.49 139.7 0))
@@
     (pin "9")
   )
-  (symbol (lib_id "74xx:74HC14") (at 109.22 86.36 0)
+  (symbol (lib_id "74xx:74HC14") (at 109.22 86.36 0) (unit 2)
     (in_bom yes) (on_board yes) (fields_autoplaced)
     (property "Reference" "U2" (id 0) (at 109.22 77.47 0))
@@
     (pin "4")
   )
-  (symbol (lib_id "Device:C") (at 97.79 58.42 0)
+  (symbol (lib_id "Device:C") (at 97.79 58.42 0) (unit 1)
     (in_bom yes) (on_board yes) (fields_autoplaced)
     (property "Reference" "C3" (id 0) (at 101.6 57.1499 0)
@@
     (pin "2")
   )
-  (symbol (lib_id "power:+3.3V") (at 81.28 68.58 0)
+  (symbol (lib_id "power:+3.3V") (at 81.28 68.58 0) (unit 1)
     (in_bom yes) (on_board yes) (fields_autoplaced)
     (property "Reference" "#PWR019" (id 0) (at 81.28 72.39 0)
@@
     (pin "1")
   )
-  (symbol (lib_id "power:+3.3V") (at 165.1 115.57 0)
+  (symbol (lib_id "power:+3.3V") (at 165.1 115.57 0) (unit 1)
     (in_bom yes) (on_board yes) (fields_autoplaced)
     (property "Reference" "#PWR026" (id 0) (at 165.1 119.38 0)
@@
     (pin "1")
   )
-  (symbol (lib_id "Device:R") (at 81.28 140.97 180)
+  (symbol (lib_id "Device:R") (at 81.28 140.97 180) (unit 1)
     (in_bom yes) (on_board yes) (fields_autoplaced)
     (property "Reference" "R29" (id 0) (at 83.82 139.6999 0)
@@
     (pin "2")
   )
-  (symbol (lib_id "power:+3.3V") (at 81.28 130.81 0)
+  (symbol (lib_id "power:+3.3V") (at 81.28 130.81 0) (unit 1)
     (in_bom yes) (on_board yes) (fields_autoplaced)
     (property "Reference" "#PWR021" (id 0) (at 81.28 134.62 0)
@@
     (pin "1")
   )
-  (symbol (lib_id "Device:C") (at 99.06 124.46 0)
+  (symbol (lib_id "Device:C") (at 99.06 124.46 0) (unit 1)
     (in_bom yes) (on_board yes) (fields_autoplaced)
     (property "Reference" "C5" (id 0) (at 102.87 123.1899 0)
@@
     (pin "2")
   )
-  (symbol (lib_id "74xx:74HC14") (at 109.22 50.8 0)
+  (symbol (lib_id "74xx:74HC14") (at 109.22 50.8 0) (unit 1)
     (in_bom yes) (on_board yes) (fields_autoplaced)
     (property "Reference" "U2" (id 0) (at 109.22 41.91 0))
@@
     (pin "2")
   )
-  (symbol (lib_id "Device:C") (at 99.06 93.98 0)
+  (symbol (lib_id "Device:C") (at 99.06 93.98 0) (unit 1)
     (in_bom yes) (on_board yes) (fields_autoplaced)
     (property "Reference" "C4" (id 0) (at 102.87 92.7099 0)
@@
     (pin "2")
   )
-  (symbol (lib_id "power:+3.3V") (at 168.91 29.21 0)
+  (symbol (lib_id "power:+3.3V") (at 168.91 29.21 0) (unit 1)
     (in_bom yes) (on_board yes) (fields_autoplaced)
     (property "Reference" "#PWR028" (id 0) (at 168.91 33.02 0)
@@
     (pin "1")
   )
-  (symbol (lib_id "Device:R") (at 81.28 109.22 180)
+  (symbol (lib_id "Device:R") (at 81.28 109.22 180) (unit 1)
     (in_bom yes) (on_board yes) (fields_autoplaced)
     (property "Reference" "R28" (id 0) (at 83.82 107.9499 0)
@@
     (pin "2")
   )
-  (symbol (lib_id "Device:R") (at 179.07 82.55 90)
+  (symbol (lib_id "Device:R") (at 179.07 82.55 90) (unit 1)
     (in_bom yes) (on_board yes) (fields_autoplaced)
     (property "Reference" "R37" (id 0) (at 179.07 76.2 90))
@@
     (pin "2")
   )
-  (symbol (lib_id "Device:R") (at 91.44 116.84 90)
+  (symbol (lib_id "Device:R") (at 91.44 116.84 90) (unit 1)
     (in_bom yes) (on_board yes) (fields_autoplaced)
     (property "Reference" "R32" (id 0) (at 91.44 110.49 90))

Commit message: Corrigido o footprint dos capacitores. Adicionado um capacitor de bypass. Adicionado o ground plane e logo.
Parts:
- added C9: 10uF, Capacitor_THT:CP_Radial_D4.0mm_P2.00mm, symbol Device:C_Polarized
- C3, C4, C5, C6, C7, C8: footprint Capacitor_THT:C_Rect_L4.6mm_W3.0mm_P2.50mm_MKS02_FKP02 -> Capacitor_THT:C_Rect_L7.0mm_W3.5mm_P5.00mm
Connections:
- net +3V3: now also C9.1
- net GND: now also C9.2
Changed lines of the file:
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@@
   (junction (at 81.28 148.59) (diameter 0) (color 0 0 0 0)
   )
+  (junction (at 165.1 118.11) (diameter 0) (color 0 0 0 0)
+  )
+  (junction (at 165.1 147.32) (diameter 0) (color 0 0 0 0)
+  )
   (junction (at 186.69 46.99) (diameter 0) (color 0 0 0 0)
   )
@@
     (stroke (width 0) (type default) (color 0 0 0 0))
   )
+  (wire (pts (xy 165.1 147.32) (xy 165.1 151.13))
+    (stroke (width 0) (type default) (color 0 0 0 0))
+  )
+  (wire (pts (xy 184.15 147.32) (xy 165.1 147.32))
+    (stroke (width 0) (type default) (color 0 0 0 0))
+  )
   (wire (pts (xy 99.06 86.36) (xy 99.06 90.17))
     (stroke (width 0) (type default) (color 0 0 0 0))
@@
     (stroke (width 0) (type default) (color 0 0 0 0))
   )
+  (wire (pts (xy 184.15 119.38) (xy 184.15 118.11))
+    (stroke (width 0) (type default) (color 0 0 0 0))
+  )
   (wire (pts (xy 118.11 148.59) (xy 124.46 148.59))
     (stroke (width 0) (type default) (color 0 0 0 0))
@@
     (stroke (width 0) (type default) (color 0 0 0 0))
   )
-  (wire (pts (xy 165.1 146.05) (xy 165.1 151.13))
-    (stroke (width 0) (type default) (color 0 0 0 0))
-  )
-  (wire (pts (xy 165.1 115.57) (xy 165.1 120.65))
+  (wire (pts (xy 165.1 146.05) (xy 165.1 147.32))
+    (stroke (width 0) (type default) (color 0 0 0 0))
+  )
+  (wire (pts (xy 165.1 115.57) (xy 165.1 118.11))
     (stroke (width 0) (type default) (color 0 0 0 0))
   )
@@
     (stroke (width 0) (type default) (color 0 0 0 0))
   )
+  (wire (pts (xy 184.15 118.11) (xy 165.1 118.11))
+    (stroke (width 0) (type default) (color 0 0 0 0))
+  )
   (wire (pts (xy 99.06 97.79) (xy 99.06 101.6))
     (stroke (width 0) (type default) (color 0 0 0 0))
@@
     (stroke (width 0) (type default) (color 0 0 0 0))
   )
+  (wire (pts (xy 184.15 127) (xy 184.15 147.32))
+    (stroke (width 0) (type default) (color 0 0 0 0))
+  )
   (wire (pts (xy 99.06 148.59) (xy 102.87 148.59))
     (stroke (width 0) (type default) (color 0 0 0 0))
@@
   )
   (wire (pts (xy 186.69 46.99) (xy 195.58 46.99))
+    (stroke (width 0) (type default) (color 0 0 0 0))
+  )
+  (wire (pts (xy 165.1 118.11) (xy 165.1 120.65))
     (stroke (width 0) (type default) (color 0 0 0 0))
   )
@@
       (effects (font (size 1.27 1.27)) (justify left))
     )
-    (property "Footprint" "Capacitor_THT:C_Rect_L4.6mm_W3.0mm_P2.50mm_MKS02_FKP02" (id 2) (at 187.6552 58.42 0)
+    (property "Footprint" "Capacitor_THT:C_Rect_L7.0mm_W3.5mm_P5.00mm" (id 2) (at 187.6552 58.42 0)
       (effects (font (size 1.27 1.27)) hide)
     )
@@
       (effects (font (size 1.27 1.27)) (justify left))
     )
-    (property "Footprint" "Capacitor_THT:C_Rect_L4.6mm_W3.0mm_P2.50mm_MKS02_FKP02" (id 2) (at 187.6552 93.98 0)
+    (property "Footprint" "Capacitor_THT:C_Rect_L7.0mm_W3.5mm_P5.00mm" (id 2) (at 187.6552 93.98 0)
       (effects (font (size 1.27 1.27)) hide)
     )
@@
       (effects (font (size 1.27 1.27)) (justify left))
     )
-    (property "Footprint" "Capacitor_THT:C_Rect_L4.6mm_W3.0mm_P2.50mm_MKS02_FKP02" (id 2) (at 100.0252 160.02 0)
+    (property "Footprint" "Capacitor_THT:C_Rect_L7.0mm_W3.5mm_P5.00mm" (id 2) (at 100.0252 160.02 0)
       (effects (font (size 1.27 1.27)) hide)
     )
@@
       (effects (font (size 1.27 1.27)) (justify left))
     )
-    (property "Footprint" "Capacitor_THT:C_Rect_L4.6mm_W3.0mm_P2.50mm_MKS02_FKP02" (id 2) (at 98.7552 62.23 0)
+    (property "Footprint" "Capacitor_THT:C_Rect_L7.0mm_W3.5mm_P5.00mm" (id 2) (at 98.7552 62.23 0)
       (effects (font (size 1.27 1.27)) hide)
     )
@@
       (effects (font (size 1.27 1.27)) (justify left))
     )
-    (property "Footprint" "Capacitor_THT:C_Rect_L4.6mm_W3.0mm_P2.50mm_MKS02_FKP02" (id 2) (at 100.0252 128.27 0)
+    (property "Footprint" "Capacitor_THT:C_Rect_L7.0mm_W3.5mm_P5.00mm" (id 2) (at 100.0252 128.27 0)
       (effects (font (size 1.27 1.27)) hide)
     )
@@
       (effects (font (size 1.27 1.27)) (justify left))
     )
-    (property "Footprint" "Capacitor_THT:C_Rect_L4.6mm_W3.0mm_P2.50mm_MKS02_FKP02" (id 2) (at 100.0252 97.79 0)
+    (property "Footprint" "Capacitor_THT:C_Rect_L7.0mm_W3.5mm_P5.00mm" (id 2) (at 100.0252 97.79 0)
       (effects (font (size 1.27 1.27)) hide)
     )
@@
       (effects (font (size 1.27 1.27)) hide)
     )
+    (pin "1")
+    (pin "2")
+  )
+  (symbol (lib_id "Device:C_Polarized") (at 184.15 123.19 0) (unit 1)
+    (in_bom yes) (on_board yes) (fields_autoplaced)
+    (property "Reference" "C9" (id 0) (at 187.96 121.0309 0)
+      (effects (font (size 1.27 1.27)) (justify left))
+    )
+    (property "Value" "10uF" (id 1) (at 187.96 123.5709 0)
+      (effects (font (size 1.27 1.27)) (justify left))
+    )
+    (property "Footprint" "Capacitor_THT:CP_Radial_D4.0mm_P2.00mm" (id 2) (at 185.1152 127 0)
+      (effects (font (size 1.27 1.27)) hide)
+    )
+    (property "Datasheet" "~" (id 3) (at 184.15 123.19 0)
+      (effects (font (size 1.27 1.27)) hide)
+    )

Commit message: Corrigido o botão de seleção de Clock e valores dos capacitores.
Parts:
- C3, C4, C5, C6, C7, C8: value 100nF -> 47nF
Changed lines of the file:
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@@
       (effects (font (size 1.27 1.27)) (justify left))
     )
-    (property "Value" "100nF" (id 1) (at 190.5 55.8799 0)
+    (property "Value" "47nF" (id 1) (at 190.5 55.8799 0)
       (effects (font (size 1.27 1.27)) (justify left))
     )
@@
       (effects (font (size 1.27 1.27)) (justify left))
     )
-    (property "Value" "100nF" (id 1) (at 190.5 91.4399 0)
+    (property "Value" "47nF" (id 1) (at 190.5 91.4399 0)
       (effects (font (size 1.27 1.27)) (justify left))
     )
@@
       (effects (font (size 1.27 1.27)) (justify left))
     )
-    (property "Value" "100nF" (id 1) (at 102.87 157.4799 0)
+    (property "Value" "47nF" (id 1) (at 102.87 157.4799 0)
       (effects (font (size 1.27 1.27)) (justify left))
     )
@@
       (effects (font (size 1.27 1.27)) (justify left))
     )
-    (property "Value" "100nF" (id 1) (at 101.6 59.6899 0)
+    (property "Value" "47nF" (id 1) (at 101.6 59.6899 0)
       (effects (font (size 1.27 1.27)) (justify left))
     )
@@
       (effects (font (size 1.27 1.27)) (justify left))
     )
-    (property "Value" "100nF" (id 1) (at 102.87 125.7299 0)
+    (property "Value" "47nF" (id 1) (at 102.87 125.7299 0)
       (effects (font (size 1.27 1.27)) (justify left))
     )
@@
       (effects (font (size 1.27 1.27)) (justify left))
     )
-    (property "Value" "100nF" (id 1) (at 102.87 95.2499 0)
-      (effects (font (size 1.27 1.27)) (justify left))
-    )
+    (property "Value" "47nF" (id 1) (at 102.87 95.2499 0)
+      (effects (font (size 1.27 1.27)) (justify left))
+    )

Commit message: Atualizado os valores dos capacitores
Parts:
- C3, C4, C5, C6, C7, C8: value 47nF -> 100nF
Changed lines of the file:
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@@
       (effects (font (size 1.27 1.27)) (justify left))
     )
-    (property "Value" "47nF" (id 1) (at 190.5 55.8799 0)
+    (property "Value" "100nF" (id 1) (at 190.5 55.8799 0)
       (effects (font (size 1.27 1.27)) (justify left))
     )
@@
       (effects (font (size 1.27 1.27)) (justify left))
     )
-    (property "Value" "47nF" (id 1) (at 190.5 91.4399 0)
+    (property "Value" "100nF" (id 1) (at 190.5 91.4399 0)
       (effects (font (size 1.27 1.27)) (justify left))
     )
@@
       (effects (font (size 1.27 1.27)) (justify left))
     )
-    (property "Value" "47nF" (id 1) (at 102.87 157.4799 0)
+    (property "Value" "100nF" (id 1) (at 102.87 157.4799 0)
       (effects (font (size 1.27 1.27)) (justify left))
     )
@@
       (effects (font (size 1.27 1.27)) (justify left))
     )
-    (property "Value" "47nF" (id 1) (at 101.6 59.6899 0)
+    (property "Value" "100nF" (id 1) (at 101.6 59.6899 0)
       (effects (font (size 1.27 1.27)) (justify left))
     )
@@
       (effects (font (size 1.27 1.27)) (justify left))
     )
-    (property "Value" "47nF" (id 1) (at 102.87 125.7299 0)
+    (property "Value" "100nF" (id 1) (at 102.87 125.7299 0)
       (effects (font (size 1.27 1.27)) (justify left))
     )
@@
       (effects (font (size 1.27 1.27)) (justify left))
     )
-    (property "Value" "47nF" (id 1) (at 102.87 95.2499 0)
-      (effects (font (size 1.27 1.27)) (justify left))
-    )
+    (property "Value" "100nF" (id 1) (at 102.87 95.2499 0)
+      (effects (font (size 1.27 1.27)) (justify left))
+    )
